Commit message: Temp moveit2 config

File: GenericHRLoader/urdf/h1.urdf (robot description, URDF)
Before this commit: robot h1_description, 25 links, 24 joints
Links:
- link logo_link: geometry collision sphere radius=0.001; visual mesh filename=file:///home/aurum/RosProjects/HRCSandbox/src/GenericHRLoad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
Joints:
- joint left_ankle_joint: limit lower=-0.87 upper=0.52 effort=40 velocity=9 -> lower=-0.87 upper=0.52 effort=40.0 velocity=9.0
- joint left_elbow_joint: limit lower=-1.25 upper=2.61 effort=18 velocity=20 -> lower=-1.25 upper=2.61 effort=18.0 velocity=20.0
- joint left_hip_pitch_joint: limit lower=-3.14 upper=2.53 effort=200 velocity=23 -> lower=-3.14 upper=2.53 effort=200.0 velocity=23.0
- joint left_hip_roll_joint: limit lower=-0.43 upper=0.43 effort=200 velocity=23 -> lower=-0.43 upper=0.43 effort=200.0 velocity=23.0
- joint left_hip_yaw_joint: limit lower=-0.43 upper=0.43 effort=200 velocity=23 -> lower=-0.43 upper=0.43 effort=200.0 velocity=23.0
- joint left_knee_joint: limit lower=-0.26 upper=2.05 effort=300 velocity=14 -> lower=-0.26 upper=2.05 effort=300.0 velocity=14.0
- joint left_shoulder_pitch_joint: limit lower=-2.87 upper=2.87 effort=40 velocity=9 -> lower=-2.87 upper=2.87 effort=40.0 velocity=9.0
- joint left_shoulder_roll_joint: limit lower=-0.34 upper=3.11 effort=40 velocity=9 -> lower=-0.34 upper=3.11 effort=40.0 velocity=9.0
- joint left_shoulder_yaw_joint: limit lower=-1.3 upper=4.45 effort=18 velocity=20 -> lower=-1.3 upper=4.45 effort=18.0 velocity=20.0
- joint right_ankle_joint: limit lower=-0.87 upper=0.52 effort=40 velocity=9 -> lower=-0.87 upper=0.52 effort=40.0 velocity=9.0
- joint right_elbow_joint: limit lower=-1.25 upper=2.61 effort=18 velocity=20 -> lower=-1.25 upper=2.61 effort=18.0 velocity=20.0
- joint right_hip_pitch_joint: limit lower=-3.14 upper=2.53 effort=200 velocity=23 -> lower=-3.14 upper=2.53 effort=200.0 velocity=23.0
- joint right_hip_roll_joint: limit lower=-0.43 upper=0.43 effort=200 velocity=23 -> lower=-0.43 upper=0.43 effort=200.0 velocity=23.0
- joint right_hip_yaw_joint: limit lower=-0.43 upper=0.43 effort=200 velocity=23 -> lower=-0.43 upper=0.43 effort=200.0 velocity=23.0
- joint right_knee_joint: limit lower=-0.26 upper=2.05 effort=300 velocity=14 -> lower=-0.26 upper=2.05 effort=300.0 velocity=14.0
- joint right_shoulder_pitch_joint: limit lower=-2.87 upper=2.87 effort=40 velocity=9 -> lower=-2.87 upper=2.87 effort=40.0 velocity=9.0
- joint right_shoulder_roll_joint: limit lower=-3.11 upper=0.34 effort=40 velocity=9 -> lower=-3.11 upper=0.34 effort=40.0 velocity=9.0
- joint right_shoulder_yaw_joint: limit lower=-4.45 upper=1.3 effort=18 velocity=20 -> lower=-4.45 upper=1.3 effort=18.0 velocity=20.0
- joint torso_joint: limit lower=-2.35 upper=2.35 effort=200 velocity=23 -> lower=-2.35 upper=2.35 effort=200.0 velocity=23.0
